File: rpi-cm4-csi-adapter.kicad_pcb (KiCad board)
At the start: 4 copper layers, 47 x 33 mm, 19 parts, among them J1 687122149022, J2 WE_68715014522

Commit message: Generate local libraries
Parts:
- D1: footprint antmicro-footprints:LED_0603 -> rpi-cm4-csi-adapter-footprints:LED_0603
- J2: footprint antmicro-footprints:WE_68715014522 -> rpi-cm4-csi-adapter-footprints:WE_68715014522
- N1: footprint antmicro-footprints:antmicro-logo_scaled_12mm -> rpi-cm4-csi-adapter-footprints:antmicro-logo_scaled_12mm
- N2: footprint antmicro-footprints:oshw-logo -> rpi-cm4-csi-adapter-footprints:oshw-logo
- R1, R2, R3: footprint antmicro-footprints:0402-res -> rpi-cm4-csi-adapter-footprints:0402-res
- TP1, TP2, TP3, TP4, TP5, TP6, TP7: footprint antmicro-footprints:TP-R-1.5 -> rpi-cm4-csi-adapter-footprints:TP-R-1.5
Changed lines of the file:
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@@
     (add_net /CAM1_D3_P)
   )
-  (module antmicro-footprints:TP-R-1.5 (layer F.Cu)
+  (module rpi-cm4-csi-adapter-footprints:TP-R-1.5 (layer F.Cu)
     (at 190.5 64.5)
     (attr virtual)
@@
       (net 38 /CAM_GPIO))
   )
-  (module antmicro-footprints:0402-res (layer F.Cu)
+  (module rpi-cm4-csi-adapter-footprints:0402-res (layer F.Cu)
     (at 196 80 270)
     (descr "Resistor SMD 0402 (1005 Metric), square (rectangular) end terminal, IPC_7351 nominal, (Body size source: http://www.tortai-tech.com/upload/download/2011102023233369053.pdf), generated with kicad-footprint-generator")
@@
     (pad 1 smd roundrect (at -0.485 0 270) (size 0.59 0.64) (layers F.Cu F.Paste F.Mask) (roundrect_rratio 0.25)
       (net 49 "Net-(D1-Pad2)"))
-    (model ${ANT3DMDL}/0402-res.step
+    (model ${KIPRJMOD}/lib/3d-models/0402-res.step
       (offset (xyz 0 0 -0.01))
       (scale (xyz 1 1 1))
@@
     )
   )
-  (module antmicro-footprints:LED_0603 (layer F.Cu)
+  (module rpi-cm4-csi-adapter-footprints:LED_0603 (layer F.Cu)
     (at 196 77.5 90)
     (attr smd)
@@
     (pad 2 smd rect (at -0.75 0 90) (size 0.8 0.8) (layers F.Cu F.Paste F.Mask)
       (net 49 "Net-(D1-Pad2)"))
-    (model ${ANT3DMDL}/LED0603.step
+    (model ${KIPRJMOD}/lib/3d-models/LED0603.step
       (at (xyz 0 0 0))
       (scale (xyz 1 1 1))
@@
     )
   )
-  (module antmicro-footprints:TP-R-1.5 (layer F.Cu)
+  (module rpi-cm4-csi-adapter-footprints:TP-R-1.5 (layer F.Cu)
     (at 197.25 69.75)
     (attr virtual)
@@
       (net 15 VCC_3V3))
   )
-  (module antmicro-footprints:TP-R-1.5 (layer F.Cu)
+  (module rpi-cm4-csi-adapter-footprints:TP-R-1.5 (layer F.Cu)
     (at 199.25 71.75)
     (attr virtual)
@@
     )
   )
-  (module antmicro-footprints:TP-R-1.5 (layer F.Cu)
+  (module rpi-cm4-csi-adapter-footprints:TP-R-1.5 (layer F.Cu)
     (at 196 66.5)
     (attr virtual)
@@
       (net 20 /SCL2))
   )
-  (module antmicro-footprints:TP-R-1.5 (layer F.Cu)
+  (module rpi-cm4-csi-adapter-footprints:TP-R-1.5 (layer F.Cu)
     (at 195 64.5)
     (attr virtual)
@@
       (net 19 /SDA2))
   )
-  (module antmicro-footprints:TP-R-1.5 (layer F.Cu)
+  (module rpi-cm4-csi-adapter-footprints:TP-R-1.5 (layer F.Cu)
     (at 193.5 71.25)
     (attr virtual)
@@
       (net 14 /RPI_SDA0))
   )
-  (module antmicro-footprints:TP-R-1.5 (layer F.Cu)
+  (module rpi-cm4-csi-adapter-footprints:TP-R-1.5 (layer F.Cu)
     (at 191.75 73)
     (attr virtual)
@@
       (net 13 /RPI_SCL0))
   )
-  (module antmicro-footprints:0402-res (layer F.Cu)
+  (module rpi-cm4-csi-adapter-footprints:0402-res (layer F.Cu)
     (at 193.5 68.25 90)
     (descr "Resistor SMD 0402 (1005 Metric), square (rectangular) end terminal, IPC_7351 nominal, (Body size source: http://www.tortai-tech.com/upload/download/2011102023233369053.pdf), generated with kicad-footprint-generator")
@@
     (pad 1 smd roundrect (at -0.485 0 90) (size 0.59 0.64) (layers F.Cu F.Paste F.Mask) (roundrect_rratio 0.25)
       (net 14 /RPI_SDA0))
-    (model ${ANT3DMDL}/0402-res.step
+    (model ${KIPRJMOD}/lib/3d-models/0402-res.step
       (offset (xyz 0 0 -0.01))
       (scale (xyz 1 1 1))
@@
     )
   )
-  (module antmicro-footprints:0402-res (layer F.Cu)
+  (module rpi-cm4-csi-adapter-footprints:0402-res (layer F.Cu)
     (at 191.75 68.25 90)
     (descr "Resistor SMD 0402 (1005 Metric), square (rectangular) end terminal, IPC_7351 nominal, (Body size source: http://www.tortai-tech.com/upload/download/2011102023233369053.pdf), generated with kicad-footprint-generator")
@@
     (pad 1 smd roundrect (at -0.485 0 90) (size 0.59 0.64) (layers F.Cu F.Paste F.Mask) (roundrect_rratio 0.25)
       (net 13 /RPI_SCL0))
-    (model ${ANT3DMDL}/0402-res.step
+    (model ${KIPRJMOD}/lib/3d-models/0402-res.step
       (offset (xyz 0 0 -0.01))
       (scale (xyz 1 1 1))
@@
     )
   )
-  (module antmicro-footprints:WE_68715014522 (layer F.Cu)
+  (module rpi-cm4-csi-adapter-footprints:WE_68715014522 (layer F.Cu)
     (at 186.2 57)
     (attr smd)
@@
     (pad 1 smd rect (at -12.25 0.6) (size 0.3 1.2) (layers F.Cu F.Paste F.Mask)
       (net 10 /CAM1_D3_N))
-    (model ${ANT3DMDL}/WE_68715014522.stp
+    (model ${KIPRJMOD}/lib/3d-models/WE_68715014522.stp
       (offset (xyz 0 -2.5 1))
       (scale (xyz 1 1 1))
@@
     )
   )
-  (module antmicro-footprints:antmicro-logo_scaled_12mm (layer F.Cu)
+  (module rpi-cm4-csi-adapter-footprints:antmicro-logo_scaled_12mm (layer F.Cu)
     (at 164.8 71.5 90)
     (attr virtual)
@@
     )
   )
-  (module antmicro-footprints:oshw-logo (layer F.Cu)
+  (module rpi-cm4-csi-adapter-footprints:oshw-logo (layer F.Cu)
     (at 205.5 70 90)
     (attr virtual)
